File: openevsetester.sch (EAGLE design)
At the start: 149 parts, among them IC1 LM321MF, Q10 BSS138, Q7 XTAL_CFPX-217

Commit message: isolated adc instead of dc/dc, op-amp and i2c isolator
Parts:
- removed C4: 10u, resistor:C-EUC0805
- removed C5: 100n, resistor:C-EUC0402
- removed C66: 100n, rcl:C-EUC0402
- removed C67: 10u, rcl:C-EUC0805
- removed IC1: LM321MF, linear:LM321MF
- removed J4: (no value), Wurth_Connectors_WR-PHD:6100XX13321_61001413321
- removed R52, R53: 0R, resistor:R-EU_R0402
- removed R54: 0k, resistor:R-EU_R0402
- removed R61: 500k, resistor:R-EU_R0402
- removed R62, R65: 1M 1% 0805 230v-safe, resistor:R-EU_R0402
- removed U$25: ISO154X, mylib:ISO154X
- removed U$37: RECOM_R0.25D-3.312, mylib:RECOM_R0.25D-3.312
- removed U$39: ESP32-S2-WROOM, mylib:ESP32-S2-WROOM
- removed U$40: MICROCHIP_MCP3021, mylib:MICROCHIP_MCP3021
- added C14: 10u, rcl:C-EUC0805
- added C15, C16: 1n, resistor:C-EUC1206
- added C17, C20: 100n, resistor:C-EUC0603
- added C18: 100n, resistor:C-EUC1206
- added C21: 1uF, resistor:C-EUC1206
- added C22: 1uF, resistor:C-EUC0603
- added C23: 1n, resistor:C-EUC0603
- added C25: 10n, resistor:C-EUC0603
- added C6: 100n, rcl:C-EUC0402
- added R72: 4k7, resistor:R-EU_R0402
- added R73: 680R, resistor:R-EU_R1210
- added U$43: OMRON_G6RL-14-ASI, mylib:OMRON_G6RL-14-ASI
- added U1: ESP32MOD, mylib:ESP32MOD
- C1, C41: device rcl:C-EUC0805 -> rcl:C-EUC0402
- R18: value 0R -> 47k
- R2: value 1k5 0,5W -> 1k5; device resistor:R-EU_R0805 -> resistor:R-EU_R1210
- R24: value 4k7 -> 10R 1% 400V; device resistor:R-EU_R0402 -> resistor:R-EU_R2512
- R25: value 4k7 -> 10R; device resistor:R-EU_R0402 -> resistor:R-EU_R2512
- R27: value 3k3 -> 237R 1% 400V; device resistor:R-EU_R0402 -> resistor:R-EU_R2010
- R28: value 10k -> 237R 1% 400V; device resistor:R-EU_R0402 -> resistor:R-EU_R2010
- R29: value 47k -> 10R; device resistor:R-EU_R0402 -> resistor:R-EU_R2512
- R3: value 220R 0,5W -> 220R; device resistor:R-EU_R0805 -> resistor:R-EU_R1210
- R4: value 680R 0,5W -> 0k; device resistor:R-EU_R0805 -> resistor:R-EU_R0402
- R7: value 4k7 0,5W -> 4k7; device resistor:R-EU_R0805 -> resistor:R-EU_R1210
- R8: value 100R 0,5W -> 100R; device resistor:R-EU_R0805 -> resistor:R-EU_R1210
- U$1, U$17, U$2, U$3, U$4, U$5, U$6, U$7: value RELAIS_MOSFET_OMRON_G3VM-351 -> IXYS_CPC1014N; device mylib:RELAIS_MOSFET_OMRON_G3VM-351 -> mylib:IXYS_CPC1014N
- U$20: value RELAIS_MOSFET_OMRON_G3VM-351 -> AMC3306M25; device mylib:RELAIS_MOSFET_OMRON_G3VM-351 -> mylib:AMC3306M25
- U$9: value OMRON_G5RL-U1-E-DC3 -> IXYS_CPC1014N; device mylib:OMRON_G5RL-U1-E-DC3 -> mylib:IXYS_CPC1014N
Connections:
- removed net +5V_ISOLATED: C4.1, C5.1, IC1.V+, R24.1, R25.1, U$25.VCC1, U$37.VOUT1, U$40.VDD
- removed net -5V_ISOLATED: IC1.V-, R28.2, U$37.VOUT2
- removed net DISPLAY1: U$39.IO45
- removed net DISPLAY3: U$39.IO42
- removed net GND: C1.2, C10.2, C11.2, C12.2, C13.2, C19.2, C2.2, C24.2, C3.1, C41.2, C63.2, C66.2, C67.2, C7.2, C8.2, C9.2, J1.2, J3.1, J4.2, LED1.C, LED13.C, LED15.C, LED16.C, LED2.C, LED3.C, LED4.C, LED5.C, LED6.C, Q10.S, R10.1, R13.1, R16.1, R20.1, R22.1, R34.2, R38.2, R40.1, R43.1, R46.1, R50.1, R56.2, R57.2, R64.2, R68.2, R69.1, R70.2, U$1.A2, U$12.2, U$12.C, U$17.A2, U$18.GND, U$2.A2, U$20.A2, U$25.GND2, U$3.A2, U$35.7, U$36.GND, U$36.PGND, U$37.-VIN, U$39.GND, U$4.A2, U$41.GND, U$42.GND, U$5.A2, U$6.A2, U$7.A2
- removed net LCD_CS: J4.3, U$39.IO14
- removed net LCD_DC: J4.5, U$39.IO16
- removed net LCD_LED: J4.8, U$39.IO21
- removed net LCD_MISO: J4.9, R53.2, U$39.IO26
- removed net LCD_MOSI: J4.6, R18.1, U$39.IO17
- removed net LCD_RESET: J4.4, U$39.IO15
- removed net LCD_SCK: J4.7, R52.1, U$39.IO18
- removed net N$24: IC1.-IN, R27.2, R28.1, R29.1
- removed net N$27: IC1.OUT, R27.1, U$40.VIN+
- removed net N$28: R24.2, U$25.SDA1, U$40.SDL
- removed net N$29: R25.2, U$25.SCL1, U$40.SCL
- removed net N$45: R29.2, R61.2, R62.1, U$34.+VOUT
- removed net TOUCH_CLK: J4.10, R52.2
- removed net TOUCH_CS: J4.11, U$39.IO35
- removed net TOUCH_D0: J4.13, R53.1
- removed net TOUCH_DIN: J4.12, R18.2
- removed net TOUCH_IRQ: J4.14, U$39.IO41
- new net AAA: C1.2, C10.2, C11.2, C12.2, C13.2, C14.2, C15.1, C17.2, C19.2, C2.2, C21.1, C24.2, C3.1, C41.2, C6.2, C63.2, C7.2, C8.2, C9.2, J1.2, J3.1, LED1.C, LED13.C, LED15.C, LED16.C, LED2.C, LED3.C, LED4.C, LED5.C, LED6.C, Q10.S, R10.1, R13.1, R16.1, R20.1, R22.1, R34.2, R38.2, R40.1, R43.1, R46.1, R50.1, R56.2, R57.2, R64.2, R68.2, R69.1, R70.2, U$1.A2, U$12.2, U$12.C, U$12.GND, U$17.A2, U$18.GND, U$2.A2, U$20.DCDC_GND, U$20.GND, U$3.A2, U$35.7, U$36.GND, U$36.PGND, U$4.A2, U$41.GND, U$42.GND, U$5.A2, U$6.A2, U$7.A2, U$9.A2, U1.GND, U1.GND@0, U1.GND@1, U1.GND@3
- new net ADC_CLKIN: U$20.CLKIN, U1.IO27
- new net ADC_DIAG: R18.1, U$20.DIAG
- new net ADC_DOUT: U$20.DOUT, U1.IO14
- new net N$37: C17.1, U$20.DCDC_IN, U$20.LDO_OUT
- new net N$42: C25.1, R25.1, U$20.INP
- new net N$49: C25.2, R29.1, U$20.INN
- new net N$50: C16.1, C18.1, C20.1, C22.2, C23.2, R24.1, R28.2, R29.2, U$20.DCDC_HGND, U$20.HGND, U$34.+VOUT
- new net N$52: C16.2, C18.2, U$20.HLDO_OUT
- new net N$54: C20.2, C22.1, C23.1, U$20.DCDC_OUT, U$20.HLDO_IN
- net +3V3: now also C15.2, C21.2, R18.2, U$20.VDD, U$43.A1, U$8.D; no longer J4.1, R5.1, R6.1, U$25.VCC2, U$37.+VIN, U$8.S, U$9.A1
- net +3V3_PERMANENT: now also R4.2, R5.1, R6.1, R72.1, U$8.S; no longer R54.2, U$8.D
- net CP: now also R27.2, U$17.S1, U$5.Q1; no longer R65.1, U$5.S1, U$6.Q1
- net EN: now also U1.EN; no longer U$39.EN
- net ESP32_VCC: now also C14.1, C6.1, R4.1, U1.VCC; no longer C66.1, C67.1, R54.1, U$39.VCC
- net GPIO0: now also U1.IO0; no longer U$39.IO0
- net GPIO_3V3_SWITCH: now also U1.IO12; no longer U$39.IO46
- net GPIO_L1: now also U1.IO32; no longer U$39.IO1
- net GPIO_L2: now also U1.IO25; no longer U$39.IO2
- net GPIO_L3: now also U1.IO26; no longer U$39.IO3
- net GPIO_PE_BREAKER: now also U1.IO18; no longer U$39.IO36
- net GPIO_PP1: now also U1.IO5; no longer U$39.IO7
- net GPIO_PP2: now also U1.IO4; no longer U$39.IO8
- net GPIO_PP3: now also U1.IO16; no longer U$39.IO9
- net GPIO_PP4: now also U1.IO17; no longer U$39.IO10
- net GPIO_PP5: no longer U$39.IO11
- net GPIO_ROTARY_A: now also U1.SENSOR_VN; no longer U$39.IO4
- net GPIO_ROTARY_B: now also U1.IO35; no longer U$39.IO5
- net GPIO_ROTARY_BUTTON: now also R72.2, U1.SENSOR_VP; no longer U$39.IO6
- net GPIO_RTC: no longer U$39.IO12
- net GPIO_STATE_AB: now also U1.IO19; no longer U$39.IO37
- net GPIO_STATE_C: now also U1.IO21; no longer U$39.IO38
- net GPIO_STATE_D_FAULT: now also U1.IO22; no longer U$39.IO39
- net GPIO_STATE_E: now also U1.IO23; no longer U$39.IO40
- net N$14: now also U$43.A2; no longer U$9.A2
- net N$16: now also U$9.A1; no longer U$17.A1
- net N$19: now also U$17.A1; no longer U$5.A1
- net N$20: now also U$5.A1; no longer U$6.A1
- net N$26: now also U$5.S1, U$6.Q1; no longer U$20.Q1, U$6.S1
- net N$31: now also U$6.A1; no longer U$20.A1
- net N$48: now also R24.2, R25.2, R27.1; no longer IC1.+IN, R61.1, R65.2
- net PE: now also R28.1, U$17.Q1, U$43.P1, U$9.S1; no longer C4.2, C5.2, R62.2, U$17.S1, U$25.GND1, U$37.0V, U$40.VSS, U$5.Q1, U$9.P1
- net PE_IN: now also U$43.S1; no longer U$9.S1
- net PP: now also R73.2; no longer R4.2
- net PP1: now also U$9.Q1; no longer U$17.Q1
- net PP3: now also R73.1; no longer R4.1
- net PP7: now also U$6.S1; no longer U$20.S1
- net RXD: now also U1.RXD0; no longer U$39.TXD0
- net SCL: now also U1.IO33; no longer U$25.SCL2, U$39.IO33
- net SDA: now also U1.IO34; no longer U$25.SDA2, U$39.IO34
- net TXD: now also U1.TXD0; no longer U$39.RXD0
- net USB_D+: no longer U$39.IO20
- net USB_D-: no longer U$39.IO19
Other:
- note added: "100R 63A"
- note added: "1500R 13A"
- note added: "220R 32A"
- note added: "59R PP too high out of Spec PP1||PP2||,,||PP5 all PPs parallel"
- note added: "680R 20A"
- note added: "IXYSCPC1002N: 0,55R RdsOn"
- note added: "PP too low out of Spec"
- note removed: "display: spi tft"
- note removed: "todo: reduce resistors by 30? ohm as mosfet rds is about 30ohm (depending on temperature, output current, ..)"
